File: project/FPGA.kicad_sch (KiCad schematic)
At the start: 54 parts, among them J4 Conn_02x05_Odd_Even, J5 Conn_02x27_Counter_Clockwise, J6 Conn_02x27_Counter_Clockwise, U11 AMS1117-3.3, U12 AMS1117-2.5, U13 AMS1117, U15 EPCS16SI8N, U16 EP4CE6, X1 ASE-xxxMHz

Commit message: еще одни дополнения
Parts:
- renumbered U15 to U14, U16 to U15
Changed lines of the file:
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@@
   (symbol (lib_id "FPGA_Altera:EP4CE6") (at 482.6 287.02 0) (unit 4)
     (in_bom yes) (on_board yes)
-    (property "Reference" "U16" (id 0) (at 482.6 265.43 0))
+    (property "Reference" "U15" (id 0) (at 482.6 265.43 0))
     (property "Value" "EP4CE6" (id 1) (at 482.6 267.97 0))
     (property "Footprint" "Package_QFP:TQFP-144_20x20mm_P0.5mm" (id 2) (at 482.6 270.51 0)
@@
   (symbol (lib_id "power:GND") (at 523.24 528.32 0) (unit 1)
     (in_bom yes) (on_board yes) (fields_autoplaced)
-    (property "Reference" "#PWR058" (id 0) (at 523.24 534.67 0)
+    (property "Reference" "#PWR059" (id 0) (at 523.24 534.67 0)
       (effects (font (size 1.27 1.27)) hide)
     )
@@
   (symbol (lib_id "power:GND") (at 264.16 226.06 0) (unit 1)
     (in_bom yes) (on_board yes) (fields_autoplaced)
-    (property "Reference" "#PWR044" (id 0) (at 264.16 232.41 0)
+    (property "Reference" "#PWR045" (id 0) (at 264.16 232.41 0)
       (effects (font (size 1.27 1.27)) hide)
     )
@@
   (symbol (lib_id "FPGA_Altera:EP4CE6") (at 473.71 549.91 0) (unit 12)
     (in_bom yes) (on_board yes)
-    (property "Reference" "U16" (id 0) (at 487.68 537.21 0))
+    (property "Reference" "U15" (id 0) (at 487.68 537.21 0))
     (property "Value" "EP4CE6" (id 1) (at 487.68 539.75 0))
     (property "Footprint" "Package_QFP:TQFP-144_20x20mm_P0.5mm" (id 2) (at 473.71 533.4 0)
@@
   (symbol (lib_id "power:GND") (at 690.88 193.04 270) (unit 1)
     (in_bom yes) (on_board yes) (fields_autoplaced)
-    (property "Reference" "#PWR061" (id 0) (at 684.53 193.04 0)
+    (property "Reference" "#PWR062" (id 0) (at 684.53 193.04 0)
       (effects (font (size 1.27 1.27)) hide)
     )
@@
   (symbol (lib_id "FPGA_Altera:EP4CE6") (at 482.6 222.25 0) (unit 2)
     (in_bom yes) (on_board yes)
-    (property "Reference" "U16" (id 0) (at 482.6 210.82 0))
+    (property "Reference" "U15" (id 0) (at 482.6 210.82 0))
     (property "Value" "EP4CE6" (id 1) (at 482.6 213.36 0))
     (property "Footprint" "Package_QFP:TQFP-144_20x20mm_P0.5mm" (id 2) (at 482.6 205.74 0)
@@
   (symbol (lib_id "FPGA_Altera:EP4CE6") (at 476.25 476.25 0) (unit 10)
     (in_bom yes) (on_board yes)
-    (property "Reference" "U16" (id 0) (at 490.22 473.71 0)
+    (property "Reference" "U15" (id 0) (at 490.22 473.71 0)
       (effects (font (size 1.27 1.27)) (justify left))
     )
@@
   (symbol (lib_id "FPGA_Altera:EP4CE6") (at 482.6 198.12 0) (unit 1)
     (in_bom yes) (on_board yes) (fields_autoplaced)
-    (property "Reference" "U16" (id 0) (at 495.9747 181.61 0))
+    (property "Reference" "U15" (id 0) (at 495.9747 181.61 0))
     (property "Value" "EP4CE6" (id 1) (at 495.9747 184.15 0))
     (property "Footprint" "Package_QFP:TQFP-144_20x20mm_P0.5mm" (id 2) (at 482.6 181.61 0)
@@
   (symbol (lib_id "FPGA_Altera:EP4CE6") (at 482.6 425.45 0) (unit 8)
     (in_bom yes) (on_board yes)
-    (property "Reference" "U16" (id 0) (at 482.6 406.4 0))
+    (property "Reference" "U15" (id 0) (at 482.6 406.4 0))
     (property "Value" "EP4CE6" (id 1) (at 482.6 408.94 0))
     (property "Footprint" "Package_QFP:TQFP-144_20x20mm_P0.5mm" (id 2) (at 482.6 408.94 0)
@@
   (symbol (lib_id "FPGA_Altera:EP4CE6") (at 482.6 388.62 0) (unit 7)
     (in_bom yes) (on_board yes)
-    (property "Reference" "U16" (id 0) (at 482.6 368.3 0))
+    (property "Reference" "U15" (id 0) (at 482.6 368.3 0))
     (property "Value" "EP4CE6" (id 1) (at 482.6 370.84 0))
     (property "Footprint" "Package_QFP:TQFP-144_20x20mm_P0.5mm" (id 2) (at 482.6 372.11 0)
@@
   (symbol (lib_id "power:GND") (at 264.16 283.21 0) (unit 1)
     (in_bom yes) (on_board yes) (fields_autoplaced)
-    (property "Reference" "#PWR046" (id 0) (at 264.16 289.56 0)
+    (property "Reference" "#PWR047" (id 0) (at 264.16 289.56 0)
       (effects (font (size 1.27 1.27)) hide)
     )
@@
   (symbol (lib_id "power:GND") (at 491.49 572.77 0) (unit 1)
     (in_bom yes) (on_board yes) (fields_autoplaced)
-    (property "Reference" "#PWR0121" (id 0) (at 491.49 579.12 0)
+    (property "Reference" "#PWR058" (id 0) (at 491.49 579.12 0)
       (effects (font (size 1.27 1.27)) hide)
     )
@@
   (symbol (lib_id "FPGA_Altera:EP4CE6") (at 477.52 453.39 0) (unit 9)
     (in_bom yes) (on_board yes)
-    (property "Reference" "U16" (id 0) (at 487.68 445.77 0)
+    (property "Reference" "U15" (id 0) (at 487.68 445.77 0)
       (effects (font (size 1.27 1.27)) (justify left))
     )
@@
   (symbol (lib_id "power:GND") (at 523.24 591.82 0) (unit 1)
     (in_bom yes) (on_board yes) (fields_autoplaced)
-    (property "Reference" "#PWR060" (id 0) (at 523.24 598.17 0)
+    (property "Reference" "#PWR061" (id 0) (at 523.24 598.17 0)
       (effects (font (size 1.27 1.27)) hide)
     )
@@
   (symbol (lib_id "power:+5V") (at 246.38 237.49 0) (unit 1)
     (in_bom yes) (on_board yes) (fields_autoplaced)
-    (property "Reference" "#PWR042" (id 0) (at 246.38 241.3 0)
+    (property "Reference" "#PWR043" (id 0) (at 246.38 241.3 0)
       (effects (font (size 1.27 1.27)) hide)
     )
@@
   (symbol (lib_id "FPGA_Altera:EP4CE6") (at 476.25 521.97 0) (unit 11)
     (in_bom yes) (on_board yes) (fields_autoplaced)
-    (property "Reference" "U16" (id 0) (at 495.3397 501.65 0))
+    (property "Reference" "U15" (id 0) (at 495.3397 501.65 0))
     (property "Value" "EP4CE6" (id 1) (at 495.3397 504.19 0))
     (property "Footprint" "Package_QFP:TQFP-144_20x20mm_P0.5mm" (id 2) (at 476.25 505.46 0)
@@
   (symbol (lib_id "power:GND") (at 264.16 254 0) (unit 1)
     (in_bom yes) (on_board yes) (fields_autoplaced)
-    (property "Reference" "#PWR045" (id 0) (at 264.16 260.35 0)
+    (property "Reference" "#PWR046" (id 0) (at 264.16 260.35 0)
       (effects (font (size 1.27 1.27)) hide)
     )
@@
   (symbol (lib_id "power:+5V") (at 246.38 266.7 0) (unit 1)
     (in_bom yes) (on_board yes) (fields_autoplaced)
-    (property "Reference" "#PWR043" (id 0) (at 246.38 270.51 0)
+    (property "Reference" "#PWR044" (id 0) (at 246.38 270.51 0)
       (effects (font (size 1.27 1.27)) hide)
     )
@@
   (symbol (lib_id "FPGA_Altera:EP4CE6") (at 482.6 325.12 0) (unit 5)
     (in_bom yes) (on_board yes)
-    (property "Reference" "U16" (id 0) (at 482.6 306.07 0))
+    (property "Reference" "U15" (id 0) (at 482.6 306.07 0))
     (property "Value" "EP4CE6" (id 1) (at 482.6 308.61 0))
     (property "Footprint" "Package_QFP:TQFP-144_20x20mm_P0.5mm" (id 2) (at 482.6 308.61 0)
@@
   (symbol (lib_id "Flash:EPCS16SI8N") (at 328.93 332.74 0) (unit 1)
     (in_bom yes) (on_board yes) (fields_autoplaced)
-    (property "Reference" "U15" (id 0) (at 328.93 322.58 0))
+    (property "Reference" "U14" (id 0) (at 328.93 322.58 0))
     (property "Value" "EPCS16SI8N" (id 1) (at 328.93 325.12 0))
     (property "Footprint" "Package_SO:SOIC-8-1EP_3.9x4.9mm_P1.27mm_EP2.29x3mm" (id 2) (at 328.93 326.39 0)
@@
   (symbol (lib_id "power:GND") (at 523.24 560.07 0) (unit 1)
     (in_bom yes) (on_board yes) (fields_autoplaced)
-    (property "Reference" "#PWR059" (id 0) (at 523.24 566.42 0)
+    (property "Reference" "#PWR060" (id 0) (at 523.24 566.42 0)
       (effects (font (size 1.27 1.27)) hide)
     )
@@
   (symbol (lib_id "FPGA_Altera:EP4CE6") (at 482.6 355.6 0) (unit 6)
     (in_bom yes) (on_board yes)
-    (property "Reference" "U16" (id 0) (at 482.6 340.36 0))
+    (property "Reference" "U15" (id 0) (at 482.6 340.36 0))
     (property "Value" "EP4CE6" (id 1) (at 482.6 342.9 0))
     (property "Footprint" "Package_QFP:TQFP-144_20x20mm_P0.5mm" (id 2) (at 482.6 339.09 0)
@@
   (symbol (lib_id "FPGA_Altera:EP4CE6") (at 482.6 248.92 0) (unit 3)
     (in_bom yes) (on_board yes)
-    (property "Reference" "U16" (id 0) (at 482.6 231.14 0))
+    (property "Reference" "U15" (id 0) (at 482.6 231.14 0))
     (property "Value" "EP4CE6" (id 1) (at 482.6 233.68 0))
     (property "Footprint" "Package_QFP:TQFP-144_20x20mm_P0.5mm" (id 2) (at 482.6 232.41 0)
@@
   (symbol (lib_id "FPGA_Altera:EP4CE6") (at 477.52 575.31 0) (unit 13)
     (in_bom yes) (on_board yes) (fields_autoplaced)
-    (property "Reference" "U16" (id 0) (at 495.9747 558.8 0))
+    (property "Reference" "U15" (id 0) (at 495.9747 558.8 0))
     (property "Value" "EP4CE6" (id 1) (at 495.9747 561.34 0))
     (property "Footprint" "Package_QFP:TQFP-144_20x20mm_P0.5mm" (id 2) (at 477.52 558.8 0)
@@
   (symbol (lib_id "power:+5V") (at 246.38 209.55 0) (unit 1)
     (in_bom yes) (on_board yes) (fields_autoplaced)
-    (property "Reference" "#PWR041" (id 0) (at 246.38 213.36 0)
-      (effects (font (size 1.27 1.27)) hide)
-    )
+    (property "Reference" "#PWR042" (id 0) (at 246.38 213.36 0)
+      (effects (font (size 1.27 1.27)) hide)
+    )
