File: project/esp32.kicad_sch (KiCad schematic)
At the start: 28 parts, among them J11 Conn_02x09_Odd_Even, J12 Conn_02x09_Odd_Even, Q2 2N3904, Q3 2N3904, Q4 2N3904, SW6 SW_Push_Dual, SW7 SW_Push_Dual, U21 AMS1117-3.3, U22 CP2102N-Axx-xQFN28, U23 ESP32-WROOM-32

Commit message: еще одни дополнения
Parts:
- renumbered J11 to J10, J12 to J11, U21 to U20, U22 to U21, U23 to U22
Changed lines of the file:
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@@
   (symbol (lib_id "power:GND") (at 227.33 88.9 270) (unit 1)
     (in_bom yes) (on_board yes) (fields_autoplaced)
-    (property "Reference" "#PWR0107" (id 0) (at 220.98 88.9 0)
+    (property "Reference" "#PWR0109" (id 0) (at 220.98 88.9 0)
       (effects (font (size 1.27 1.27)) hide)
     )
@@
   (symbol (lib_id "Connector_Generic:Conn_02x09_Odd_Even") (at 201.93 100.33 0) (unit 1)
     (in_bom yes) (on_board yes) (fields_autoplaced)
-    (property "Reference" "J11" (id 0) (at 203.2 83.82 0))
+    (property "Reference" "J10" (id 0) (at 203.2 83.82 0))
     (property "Value" "Conn_02x09_Odd_Even" (id 1) (at 203.2 86.36 0))
     (property "Footprint" "Connector_PinSocket_2.54mm:PinSocket_2x09_P2.54mm_Vertical" (id 2) (at 201.93 100.33 0)
@@
   (symbol (lib_id "Regulator_Linear:AMS1117-3.3") (at 41.91 171.45 0) (unit 1)
     (in_bom yes) (on_board yes) (fields_autoplaced)
-    (property "Reference" "U21" (id 0) (at 41.91 163.83 0))
+    (property "Reference" "U20" (id 0) (at 41.91 163.83 0))
     (property "Value" "AMS1117-3.3" (id 1) (at 41.91 166.37 0))
     (property "Footprint" "Package_TO_SOT_SMD:SOT-223-3_TabPin2" (id 2) (at 41.91 166.37 0)
@@
   (symbol (lib_id "power:GND") (at 17.78 35.56 0) (unit 1)
     (in_bom yes) (on_board yes) (fields_autoplaced)
-    (property "Reference" "#PWR098" (id 0) (at 17.78 41.91 0)
+    (property "Reference" "#PWR0100" (id 0) (at 17.78 41.91 0)
       (effects (font (size 1.27 1.27)) hide)
     )
@@
   (symbol (lib_id "power:GND") (at 127 101.6 0) (unit 1)
     (in_bom yes) (on_board yes) (fields_autoplaced)
-    (property "Reference" "#PWR0104" (id 0) (at 127 107.95 0)
+    (property "Reference" "#PWR0106" (id 0) (at 127 107.95 0)
       (effects (font (size 1.27 1.27)) hide)
     )
@@
   (symbol (lib_id "power:GND") (at 111.76 25.4 0) (unit 1)
     (in_bom yes) (on_board yes) (fields_autoplaced)
-    (property "Reference" "#PWR0103" (id 0) (at 111.76 31.75 0)
+    (property "Reference" "#PWR0105" (id 0) (at 111.76 31.75 0)
       (effects (font (size 1.27 1.27)) hide)
     )
@@
   (symbol (lib_id "Connector_Generic:Conn_02x09_Odd_Even") (at 238.76 100.33 0) (unit 1)
     (in_bom yes) (on_board yes) (fields_autoplaced)
-    (property "Reference" "J12" (id 0) (at 240.03 83.82 0))
+    (property "Reference" "J11" (id 0) (at 240.03 83.82 0))
     (property "Value" "Conn_02x09_Odd_Even" (id 1) (at 240.03 86.36 0))
     (property "Footprint" "Connector_PinSocket_2.54mm:PinSocket_2x09_P2.54mm_Vertical" (id 2) (at 238.76 100.33 0)
@@
   (symbol (lib_id "power:+5V") (at 24.13 167.64 0) (unit 1)
     (in_bom yes) (on_board yes) (fields_autoplaced)
-    (property "Reference" "#PWR099" (id 0) (at 24.13 171.45 0)
+    (property "Reference" "#PWR0101" (id 0) (at 24.13 171.45 0)
       (effects (font (size 1.27 1.27)) hide)
     )
@@
   (symbol (lib_id "power:+5V") (at 17.78 25.4 0) (unit 1)
     (in_bom yes) (on_board yes) (fields_autoplaced)
-    (property "Reference" "#PWR097" (id 0) (at 17.78 29.21 0)
+    (property "Reference" "#PWR099" (id 0) (at 17.78 29.21 0)
       (effects (font (size 1.27 1.27)) hide)
     )
@@
   (symbol (lib_id "power:GND") (at 254 90.17 90) (unit 1)
     (in_bom yes) (on_board yes) (fields_autoplaced)
-    (property "Reference" "#PWR0109" (id 0) (at 260.35 90.17 0)
+    (property "Reference" "#PWR0111" (id 0) (at 260.35 90.17 0)
       (effects (font (size 1.27 1.27)) hide)
     )
@@
   (symbol (lib_id "power:GND") (at 217.17 66.04 0) (unit 1)
     (in_bom yes) (on_board yes) (fields_autoplaced)
-    (property "Reference" "#PWR0106" (id 0) (at 217.17 72.39 0)
+    (property "Reference" "#PWR0108" (id 0) (at 217.17 72.39 0)
       (effects (font (size 1.27 1.27)) hide)
     )
@@
   (symbol (lib_id "power:GND") (at 45.72 22.86 180) (unit 1)
     (in_bom yes) (on_board yes) (fields_autoplaced)
-    (property "Reference" "#PWR0101" (id 0) (at 45.72 16.51 0)
+    (property "Reference" "#PWR0103" (id 0) (at 45.72 16.51 0)
       (effects (font (size 1.27 1.27)) hide)
     )
@@
   (symbol (lib_id "RF_Module:ESP32-WROOM-32") (at 127 63.5 0) (unit 1)
     (in_bom yes) (on_board yes) (fields_autoplaced)
-    (property "Reference" "U23" (id 0) (at 129.0194 25.4 0)
+    (property "Reference" "U22" (id 0) (at 129.0194 25.4 0)
       (effects (font (size 1.27 1.27)) (justify left))
     )
@@
   (symbol (lib_id "Interface_USB:CP2102N-Axx-xQFN28") (at 45.72 67.31 0) (unit 1)
     (in_bom yes) (on_board yes)
-    (property "Reference" "U22" (id 0) (at 47.7394 100.33 0)
+    (property "Reference" "U21" (id 0) (at 47.7394 100.33 0)
       (effects (font (size 1.27 1.27)) (justify left))
     )
@@
   (symbol (lib_id "power:GND") (at 45.72 101.6 0) (unit 1)
     (in_bom yes) (on_board yes) (fields_autoplaced)
-    (property "Reference" "#PWR0102" (id 0) (at 45.72 107.95 0)
+    (property "Reference" "#PWR0104" (id 0) (at 45.72 107.95 0)
       (effects (font (size 1.27 1.27)) hide)
     )
@@
   (symbol (lib_id "power:GND") (at 162.56 182.88 0) (unit 1)
     (in_bom yes) (on_board yes) (fields_autoplaced)
-    (property "Reference" "#PWR0105" (id 0) (at 162.56 189.23 0)
+    (property "Reference" "#PWR0107" (id 0) (at 162.56 189.23 0)
       (effects (font (size 1.27 1.27)) hide)
     )
@@
   (symbol (lib_id "power:GND") (at 252.73 66.04 0) (unit 1)
     (in_bom yes) (on_board yes) (fields_autoplaced)
-    (property "Reference" "#PWR0108" (id 0) (at 252.73 72.39 0)
+    (property "Reference" "#PWR0110" (id 0) (at 252.73 72.39 0)
       (effects (font (size 1.27 1.27)) hide)
     )
@@
   (symbol (lib_id "power:GND") (at 41.91 184.15 0) (unit 1)
     (in_bom yes) (on_board yes) (fields_autoplaced)
-    (property "Reference" "#PWR0100" (id 0) (at 41.91 190.5 0)
-      (effects (font (size 1.27 1.27)) hide)
-    )
+    (property "Reference" "#PWR0102" (id 0) (at 41.91 190.5 0)
+      (effects (font (size 1.27 1.27)) hide)
+    )
