File: project/stlink.kicad_sch (KiCad schematic)
At the start: 41 parts, among them J7 Conn_01x08_Male, Q1 2N3904, SW2 SW_Push_Dual, U17 RT9193, U18 STM32F103CBTx, Y3 8MHz

Commit message: еще одни дополнения
Parts:
- renumbered R91 to R37, R90 to R40, R43 to R41, R44 to R42, R45 to R43, R46 to R44, U17 to U16, U18 to U17
Changed lines of the file:
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@@
   (symbol (lib_id "power:GND") (at 55.88 162.56 0) (unit 1)
     (in_bom yes) (on_board yes) (fields_autoplaced)
-    (property "Reference" "#PWR067" (id 0) (at 55.88 168.91 0)
+    (property "Reference" "#PWR068" (id 0) (at 55.88 168.91 0)
       (effects (font (size 1.27 1.27)) hide)
     )
@@
   (symbol (lib_id "power:GND") (at 87.63 189.23 270) (unit 1)
     (in_bom yes) (on_board yes)
-    (property "Reference" "#PWR072" (id 0) (at 81.28 189.23 0)
+    (property "Reference" "#PWR073" (id 0) (at 81.28 189.23 0)
       (effects (font (size 1.27 1.27)) hide)
     )
@@
   (symbol (lib_id "power:GND") (at 118.11 273.05 0) (unit 1)
     (in_bom yes) (on_board yes) (fields_autoplaced)
-    (property "Reference" "#PWR074" (id 0) (at 118.11 279.4 0)
+    (property "Reference" "#PWR075" (id 0) (at 118.11 279.4 0)
       (effects (font (size 1.27 1.27)) hide)
     )
@@
   (symbol (lib_id "Device:R") (at 156.21 78.74 90) (unit 1)
     (in_bom yes) (on_board yes)
-    (property "Reference" "R43" (id 0) (at 158.75 76.2 90))
+    (property "Reference" "R41" (id 0) (at 158.75 76.2 90))
     (property "Value" "100" (id 1) (at 154.94 76.2 90))
     (property "Footprint" "Resistor_SMD:R_0603_1608Metric_Pad0.98x0.95mm_HandSolder" (id 2) (at 156.21 80.518 90)
@@
   (symbol (lib_id "power:GND") (at 72.39 276.86 0) (unit 1)
     (in_bom yes) (on_board yes) (fields_autoplaced)
-    (property "Reference" "#PWR070" (id 0) (at 72.39 283.21 0)
+    (property "Reference" "#PWR071" (id 0) (at 72.39 283.21 0)
       (effects (font (size 1.27 1.27)) hide)
     )
@@
   (symbol (lib_id "Device:R") (at 255.27 106.68 90) (unit 1)
     (in_bom yes) (on_board yes)
-    (property "Reference" "R46" (id 0) (at 257.81 104.14 90))
+    (property "Reference" "R44" (id 0) (at 257.81 104.14 90))
     (property "Value" "1K" (id 1) (at 254 104.14 90))
     (property "Footprint" "Resistor_SMD:R_0603_1608Metric_Pad0.98x0.95mm_HandSolder" (id 2) (at 255.27 108.458 90)
@@
   (symbol (lib_id "MCU_ST_STM32F1:STM32F103CBTx") (at 77.47 77.47 0) (unit 1)
     (in_bom yes) (on_board yes) (fields_autoplaced)
-    (property "Reference" "U18" (id 0) (at 82.0294 115.57 0)
+    (property "Reference" "U17" (id 0) (at 82.0294 115.57 0)
       (effects (font (size 1.27 1.27)) (justify left))
     )
@@
   (symbol (lib_id "power:GND") (at 85.09 267.97 0) (unit 1)
     (in_bom yes) (on_board yes) (fields_autoplaced)
-    (property "Reference" "#PWR071" (id 0) (at 85.09 274.32 0)
+    (property "Reference" "#PWR072" (id 0) (at 85.09 274.32 0)
       (effects (font (size 1.27 1.27)) hide)
     )
@@
   (symbol (lib_id "power:+5V") (at 19.05 255.27 0) (unit 1)
     (in_bom yes) (on_board yes) (fields_autoplaced)
-    (property "Reference" "#PWR062" (id 0) (at 19.05 259.08 0)
+    (property "Reference" "#PWR063" (id 0) (at 19.05 259.08 0)
       (effects (font (size 1.27 1.27)) hide)
     )
@@
   (symbol (lib_id "power:+5V") (at 147.32 67.31 0) (unit 1)
     (in_bom yes) (on_board yes) (fields_autoplaced)
-    (property "Reference" "#PWR076" (id 0) (at 147.32 71.12 0)
+    (property "Reference" "#PWR077" (id 0) (at 147.32 71.12 0)
       (effects (font (size 1.27 1.27)) hide)
     )
@@
   (symbol (lib_id "power:GND") (at 147.32 88.9 0) (unit 1)
     (in_bom yes) (on_board yes) (fields_autoplaced)
-    (property "Reference" "#PWR077" (id 0) (at 147.32 95.25 0)
+    (property "Reference" "#PWR078" (id 0) (at 147.32 95.25 0)
       (effects (font (size 1.27 1.27)) hide)
     )
@@
   (symbol (lib_id "power:GND") (at 143.51 190.5 180) (unit 1)
     (in_bom yes) (on_board yes) (fields_autoplaced)
-    (property "Reference" "#PWR075" (id 0) (at 143.51 184.15 0)
+    (property "Reference" "#PWR076" (id 0) (at 143.51 184.15 0)
       (effects (font (size 1.27 1.27)) hide)
     )
@@
   (symbol (lib_id "power:GND") (at 35.56 66.04 0) (unit 1)
     (in_bom yes) (on_board yes) (fields_autoplaced)
-    (property "Reference" "#PWR065" (id 0) (at 35.56 72.39 0)
+    (property "Reference" "#PWR066" (id 0) (at 35.56 72.39 0)
       (effects (font (size 1.27 1.27)) hide)
     )
@@
   (symbol (lib_id "power:GND") (at 196.85 205.74 0) (unit 1)
     (in_bom yes) (on_board yes) (fields_autoplaced)
-    (property "Reference" "#PWR078" (id 0) (at 196.85 212.09 0)
+    (property "Reference" "#PWR079" (id 0) (at 196.85 212.09 0)
       (effects (font (size 1.27 1.27)) hide)
     )
@@
   (symbol (lib_id "Device:R") (at 196.85 191.77 0) (unit 1)
     (in_bom yes) (on_board yes) (fields_autoplaced)
-    (property "Reference" "R44" (id 0) (at 199.39 190.4999 0)
+    (property "Reference" "R42" (id 0) (at 199.39 190.4999 0)
       (effects (font (size 1.27 1.27)) (justify left))
     )
@@
   (symbol (lib_id "power:GND") (at 26.67 203.2 0) (unit 1)
     (in_bom yes) (on_board yes) (fields_autoplaced)
-    (property "Reference" "#PWR064" (id 0) (at 26.67 209.55 0)
+    (property "Reference" "#PWR065" (id 0) (at 26.67 209.55 0)
       (effects (font (size 1.27 1.27)) hide)
     )
@@
   (symbol (lib_id "power:GND") (at 72.39 118.11 0) (unit 1)
     (in_bom yes) (on_board yes) (fields_autoplaced)
-    (property "Reference" "#PWR069" (id 0) (at 72.39 124.46 0)
+    (property "Reference" "#PWR070" (id 0) (at 72.39 124.46 0)
       (effects (font (size 1.27 1.27)) hide)
     )
@@
   (symbol (lib_id "power:GND") (at 223.52 101.6 270) (unit 1)
     (in_bom yes) (on_board yes) (fields_autoplaced)
-    (property "Reference" "#PWR079" (id 0) (at 217.17 101.6 0)
+    (property "Reference" "#PWR080" (id 0) (at 217.17 101.6 0)
       (effects (font (size 1.27 1.27)) hide)
     )
@@
   (symbol (lib_id "power:GND") (at 19.05 269.24 0) (unit 1)
     (in_bom yes) (on_board yes) (fields_autoplaced)
-    (property "Reference" "#PWR063" (id 0) (at 19.05 275.59 0)
+    (property "Reference" "#PWR064" (id 0) (at 19.05 275.59 0)
       (effects (font (size 1.27 1.27)) hide)
     )
@@
   (symbol (lib_id "power:GND") (at 67.31 196.85 0) (unit 1)
     (in_bom yes) (on_board yes) (fields_autoplaced)
-    (property "Reference" "#PWR068" (id 0) (at 67.31 203.2 0)
+    (property "Reference" "#PWR069" (id 0) (at 67.31 203.2 0)
       (effects (font (size 1.27 1.27)) hide)
     )
@@
   (symbol (lib_id "Device:R") (at 148.59 187.96 0) (mirror x) (unit 1)
     (in_bom yes) (on_board yes)
-    (property "Reference" "R90" (id 0) (at 148.59 177.8 90))
+    (property "Reference" "R40" (id 0) (at 148.59 177.8 90))
     (property "Value" "22" (id 1) (at 148.59 181.61 90))
     (property "Footprint" "Resistor_SMD:R_0603_1608Metric_Pad0.98x0.95mm_HandSolder" (id 2) (at 146.812 187.96 90)
@@
   (symbol (lib_id "Device:R") (at 255.27 101.6 90) (unit 1)
     (in_bom yes) (on_board yes)
-    (property "Reference" "R45" (id 0) (at 257.81 99.06 90))
+    (property "Reference" "R43" (id 0) (at 257.81 99.06 90))
     (property "Value" "1K" (id 1) (at 254 99.06 90))
     (property "Footprint" "Resistor_SMD:R_0603_1608Metric_Pad0.98x0.95mm_HandSolder" (id 2) (at 255.27 103.378 90)
@@
   (symbol (lib_id "power:GND") (at 111.76 195.58 0) (unit 1)
     (in_bom yes) (on_board yes)
-    (property "Reference" "#PWR073" (id 0) (at 111.76 201.93 0)
+    (property "Reference" "#PWR074" (id 0) (at 111.76 201.93 0)
       (effects (font (size 1.27 1.27)) hide)
     )
@@
   (symbol (lib_id "TX0RX0:RT9193") (at 59.69 260.35 0) (unit 1)
     (in_bom yes) (on_board yes) (fields_autoplaced)
-    (property "Reference" "U17" (id 0) (at 59.69 251.46 0)
+    (property "Reference" "U16" (id 0) (at 59.69 251.46 0)
       (effects (font (size 1.524 1.524)))
     )
@@
   (symbol (lib_id "power:GND") (at 41.91 97.79 270) (unit 1)
     (in_bom yes) (on_board yes) (fields_autoplaced)
-    (property "Reference" "#PWR066" (id 0) (at 35.56 97.79 0)
+    (property "Reference" "#PWR067" (id 0) (at 35.56 97.79 0)
       (effects (font (size 1.27 1.27)) hide)
     )
@@
   (symbol (lib_id "Device:R") (at 146.05 187.96 0) (mirror x) (unit 1)
     (in_bom yes) (on_board yes)
-    (property "Reference" "R91" (id 0) (at 146.05 177.8 90))
+    (property "Reference" "R37" (id 0) (at 146.05 177.8 90))
     (property "Value" "22" (id 1) (at 146.05 181.61 90))
     (property "Footprint" "Resistor_SMD:R_0603_1608Metric_Pad0.98x0.95mm_HandSolder" (id 2) (at 144.272 187.96 90)
