File: project/stm32_ex.kicad_sch (KiCad schematic)
At the start: 40 parts, among them J13 RJ45_Amphenol_RJMG1BD3B8K1ANR, J14 USB_C_Receptacle_USB2.0, U24 KSZ8081RNA, U25 USBLC6-2P6, X2 ASE-xxxMHz

Commit message: еще одни дополнения
Parts:
- renumbered J13 to J12, J14 to J13, U24 to U23, U25 to U24
Changed lines of the file:
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@@
   (symbol (lib_id "power:GND") (at 185.42 90.17 0) (unit 1)
     (in_bom yes) (on_board yes)
-    (property "Reference" "#PWR0114" (id 0) (at 185.42 96.52 0)
+    (property "Reference" "#PWR0117" (id 0) (at 185.42 96.52 0)
       (effects (font (size 1.27 1.27)) hide)
     )
@@
   (symbol (lib_id "Connector:RJ45_Amphenol_RJMG1BD3B8K1ANR") (at 229.87 91.44 0) (unit 1)
     (in_bom yes) (on_board yes) (fields_autoplaced)
-    (property "Reference" "J13" (id 0) (at 229.87 72.39 0))
+    (property "Reference" "J12" (id 0) (at 229.87 72.39 0))
     (property "Value" "RJ45_Amphenol_RJMG1BD3B8K1ANR" (id 1) (at 229.87 74.93 0))
     (property "Footprint" "Connector_RJ:RJ45_Amphenol_RJMG1BD3B8K1ANR" (id 2) (at 229.87 73.66 0)
@@
   (symbol (lib_id "power:GND") (at 279.4 110.49 0) (unit 1)
     (in_bom yes) (on_board yes) (fields_autoplaced)
-    (property "Reference" "#PWR0118" (id 0) (at 279.4 116.84 0)
+    (property "Reference" "#PWR0121" (id 0) (at 279.4 116.84 0)
       (effects (font (size 1.27 1.27)) hide)
     )
@@
   (symbol (lib_id "power:GND") (at 124.46 125.73 0) (unit 1)
     (in_bom yes) (on_board yes) (fields_autoplaced)
-    (property "Reference" "#PWR0112" (id 0) (at 124.46 132.08 0)
+    (property "Reference" "#PWR0114" (id 0) (at 124.46 132.08 0)
       (effects (font (size 1.27 1.27)) hide)
     )
@@
   (symbol (lib_id "power:GND") (at 214.63 185.42 0) (mirror y) (unit 1)
     (in_bom yes) (on_board yes) (fields_autoplaced)
-    (property "Reference" "#PWR0116" (id 0) (at 214.63 191.77 0)
+    (property "Reference" "#PWR0119" (id 0) (at 214.63 191.77 0)
       (effects (font (size 1.27 1.27)) hide)
     )
@@
   (symbol (lib_id "power:GND") (at 187.96 149.86 270) (unit 1)
     (in_bom yes) (on_board yes) (fields_autoplaced)
-    (property "Reference" "#PWR0115" (id 0) (at 181.61 149.86 0)
+    (property "Reference" "#PWR0118" (id 0) (at 181.61 149.86 0)
       (effects (font (size 1.27 1.27)) hide)
     )
@@
   (symbol (lib_id "power:GND") (at 229.87 111.76 0) (unit 1)
     (in_bom yes) (on_board yes) (fields_autoplaced)
-    (property "Reference" "#PWR0117" (id 0) (at 229.87 118.11 0)
+    (property "Reference" "#PWR0120" (id 0) (at 229.87 118.11 0)
       (effects (font (size 1.27 1.27)) hide)
     )
@@
   (symbol (lib_id "power:GND") (at 142.24 55.88 270) (unit 1)
     (in_bom yes) (on_board yes) (fields_autoplaced)
-    (property "Reference" "#PWR0120" (id 0) (at 135.89 55.88 0)
+    (property "Reference" "#PWR0115" (id 0) (at 135.89 55.88 0)
       (effects (font (size 1.27 1.27)) hide)
     )
@@
   (symbol (lib_id "power:GND") (at 74.93 139.7 0) (unit 1)
     (in_bom yes) (on_board yes) (fields_autoplaced)
-    (property "Reference" "#PWR0110" (id 0) (at 74.93 146.05 0)
+    (property "Reference" "#PWR0112" (id 0) (at 74.93 146.05 0)
       (effects (font (size 1.27 1.27)) hide)
     )
@@
   (symbol (lib_id "power:GND") (at 152.4 110.49 0) (unit 1)
     (in_bom yes) (on_board yes) (fields_autoplaced)
-    (property "Reference" "#PWR0113" (id 0) (at 152.4 116.84 0)
+    (property "Reference" "#PWR0116" (id 0) (at 152.4 116.84 0)
       (effects (font (size 1.27 1.27)) hide)
     )
@@
   (symbol (lib_id "Power_Protection:USBLC6-2P6") (at 200.66 149.86 270) (mirror x) (unit 1)
     (in_bom yes) (on_board yes)
-    (property "Reference" "U25" (id 0) (at 200.66 135.89 90))
+    (property "Reference" "U24" (id 0) (at 200.66 135.89 90))
     (property "Value" "USBLC6-2P6" (id 1) (at 200.66 138.43 90))
     (property "Footprint" "Package_TO_SOT_SMD:SOT-666" (id 2) (at 187.96 149.86 0)
@@
   (symbol (lib_id "Connector:USB_C_Receptacle_USB2.0") (at 233.68 148.59 0) (mirror y) (unit 1)
     (in_bom yes) (on_board yes) (fields_autoplaced)
-    (property "Reference" "J14" (id 0) (at 233.68 125.73 0))
+    (property "Reference" "J13" (id 0) (at 233.68 125.73 0))
     (property "Value" "USB_C_Receptacle_USB2.0" (id 1) (at 233.68 128.27 0))
     (property "Footprint" "Connector_USB:USB_C_Receptacle_HRO_TYPE-C-31-M-12" (id 2) (at 229.87 148.59 0)
@@
   (symbol (lib_id "Interface_Ethernet:KSZ8081RNA") (at 124.46 99.06 0) (unit 1)
     (in_bom yes) (on_board yes) (fields_autoplaced)
-    (property "Reference" "U24" (id 0) (at 126.4794 124.46 0)
+    (property "Reference" "U23" (id 0) (at 126.4794 124.46 0)
       (effects (font (size 1.27 1.27)) (justify left))
     )
@@
   (symbol (lib_id "power:GND") (at 101.6 66.04 0) (unit 1)
     (in_bom yes) (on_board yes) (fields_autoplaced)
-    (property "Reference" "#PWR0111" (id 0) (at 101.6 72.39 0)
-      (effects (font (size 1.27 1.27)) hide)
-    )
+    (property "Reference" "#PWR0113" (id 0) (at 101.6 72.39 0)
+      (effects (font (size 1.27 1.27)) hide)
+    )
