File: project/stm32f407.kicad_sch (KiCad schematic)
At the start: 59 parts, among them J10 Conn_02x21_Odd_Even, J9 Conn_02x21_Odd_Even, SW3 SW_Push_Dual, SW4 SW_Push_Dual, SW5 SW_Push_Dual, U19 AMS1117-3.3, U20 STM32F407VGTx, Y4 8MHz, Y5 32.768KHz

Commit message: еще одни дополнения
Parts:
- renumbered J9 to J8, J10 to J9, R47 to R45, R48 to R46, R37 to R47, R40 to R48, U19 to U18, U20 to U19
Changed lines of the file:
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@@
   (symbol (lib_id "power:GND") (at 270.51 86.36 0) (unit 1)
     (in_bom yes) (on_board yes) (fields_autoplaced)
-    (property "Reference" "#PWR088" (id 0) (at 270.51 92.71 0)
+    (property "Reference" "#PWR090" (id 0) (at 270.51 92.71 0)
       (effects (font (size 1.27 1.27)) hide)
     )
@@
   (symbol (lib_id "power:GND") (at 74.93 173.99 0) (unit 1)
     (in_bom yes) (on_board yes) (fields_autoplaced)
-    (property "Reference" "#PWR083" (id 0) (at 74.93 180.34 0)
+    (property "Reference" "#PWR084" (id 0) (at 74.93 180.34 0)
       (effects (font (size 1.27 1.27)) hide)
     )
@@
   (symbol (lib_id "Device:R") (at 90.17 255.27 0) (unit 1)
     (in_bom yes) (on_board yes) (fields_autoplaced)
-    (property "Reference" "R47" (id 0) (at 92.71 253.9999 0)
+    (property "Reference" "R45" (id 0) (at 92.71 253.9999 0)
       (effects (font (size 1.27 1.27)) (justify left))
     )
@@
   (symbol (lib_id "Connector_Generic:Conn_02x21_Odd_Even") (at 184.15 129.54 0) (unit 1)
     (in_bom yes) (on_board yes) (fields_autoplaced)
-    (property "Reference" "J10" (id 0) (at 185.42 97.79 0))
+    (property "Reference" "J9" (id 0) (at 185.42 97.79 0))
     (property "Value" "Conn_02x21_Odd_Even" (id 1) (at 185.42 100.33 0))
     (property "Footprint" "Connector_PinHeader_2.54mm:PinHeader_2x21_P2.54mm_Vertical" (id 2) (at 184.15 129.54 0)
@@
   (symbol (lib_id "power:+5V") (at 25.4 254 0) (unit 1)
     (in_bom yes) (on_board yes) (fields_autoplaced)
-    (property "Reference" "#PWR081" (id 0) (at 25.4 257.81 0)
+    (property "Reference" "#PWR082" (id 0) (at 25.4 257.81 0)
       (effects (font (size 1.27 1.27)) hide)
     )
@@
   (symbol (lib_id "power:GND") (at 17.78 54.61 0) (unit 1)
     (in_bom yes) (on_board yes) (fields_autoplaced)
-    (property "Reference" "#PWR080" (id 0) (at 17.78 60.96 0)
+    (property "Reference" "#PWR081" (id 0) (at 17.78 60.96 0)
       (effects (font (size 1.27 1.27)) hide)
     )
@@
   (symbol (lib_id "power:GND") (at 273.05 154.94 0) (unit 1)
     (in_bom yes) (on_board yes) (fields_autoplaced)
-    (property "Reference" "#PWR089" (id 0) (at 273.05 161.29 0)
+    (property "Reference" "#PWR091" (id 0) (at 273.05 161.29 0)
       (effects (font (size 1.27 1.27)) hide)
     )
@@
   (symbol (lib_id "MCU_ST_STM32F4:STM32F407VGTx") (at 80.01 100.33 0) (unit 1)
     (in_bom yes) (on_board yes) (fields_autoplaced)
-    (property "Reference" "U20" (id 0) (at 87.1094 168.91 0)
+    (property "Reference" "U19" (id 0) (at 87.1094 168.91 0)
       (effects (font (size 1.27 1.27)) (justify left))
     )
@@
   (symbol (lib_id "power:GND") (at 347.98 86.36 0) (unit 1)
     (in_bom yes) (on_board yes) (fields_autoplaced)
-    (property "Reference" "#PWR095" (id 0) (at 347.98 92.71 0)
+    (property "Reference" "#PWR097" (id 0) (at 347.98 92.71 0)
       (effects (font (size 1.27 1.27)) hide)
     )
@@
   (symbol (lib_id "power:GND") (at 309.88 154.94 0) (unit 1)
     (in_bom yes) (on_board yes) (fields_autoplaced)
-    (property "Reference" "#PWR092" (id 0) (at 309.88 161.29 0)
+    (property "Reference" "#PWR094" (id 0) (at 309.88 161.29 0)
       (effects (font (size 1.27 1.27)) hide)
     )
@@
   (symbol (lib_id "power:GND") (at 100.33 271.78 0) (unit 1)
     (in_bom yes) (on_board yes) (fields_autoplaced)
-    (property "Reference" "#PWR085" (id 0) (at 100.33 278.13 0)
+    (property "Reference" "#PWR086" (id 0) (at 100.33 278.13 0)
       (effects (font (size 1.27 1.27)) hide)
     )
@@
   (symbol (lib_id "power:GND") (at 346.71 154.94 0) (unit 1)
     (in_bom yes) (on_board yes) (fields_autoplaced)
-    (property "Reference" "#PWR094" (id 0) (at 346.71 161.29 0)
+    (property "Reference" "#PWR096" (id 0) (at 346.71 161.29 0)
       (effects (font (size 1.27 1.27)) hide)
     )
@@
   (symbol (lib_id "power:GND") (at 383.54 154.94 0) (unit 1)
     (in_bom yes) (on_board yes) (fields_autoplaced)
-    (property "Reference" "#PWR096" (id 0) (at 383.54 161.29 0)
+    (property "Reference" "#PWR098" (id 0) (at 383.54 161.29 0)
       (effects (font (size 1.27 1.27)) hide)
     )
@@
   (symbol (lib_id "power:GND") (at 240.03 163.83 0) (unit 1)
     (in_bom yes) (on_board yes) (fields_autoplaced)
-    (property "Reference" "#PWR0122" (id 0) (at 240.03 170.18 0)
+    (property "Reference" "#PWR088" (id 0) (at 240.03 170.18 0)
       (effects (font (size 1.27 1.27)) hide)
     )
@@
   (symbol (lib_id "power:GND") (at 90.17 269.24 0) (unit 1)
     (in_bom yes) (on_board yes) (fields_autoplaced)
-    (property "Reference" "#PWR084" (id 0) (at 90.17 275.59 0)
+    (property "Reference" "#PWR085" (id 0) (at 90.17 275.59 0)
       (effects (font (size 1.27 1.27)) hide)
     )
@@
   (symbol (lib_id "Device:R") (at 214.63 251.46 90) (unit 1)
     (in_bom yes) (on_board yes) (fields_autoplaced)
-    (property "Reference" "R48" (id 0) (at 214.63 245.11 90))
+    (property "Reference" "R46" (id 0) (at 214.63 245.11 90))
     (property "Value" "47" (id 1) (at 214.63 247.65 90))
     (property "Footprint" "Resistor_SMD:R_0603_1608Metric_Pad0.98x0.95mm_HandSolder" (id 2) (at 214.63 253.238 90)
@@
   (symbol (lib_id "power:GND") (at 215.9 261.62 270) (unit 1)
     (in_bom yes) (on_board yes) (fields_autoplaced)
-    (property "Reference" "#PWR086" (id 0) (at 209.55 261.62 0)
+    (property "Reference" "#PWR087" (id 0) (at 209.55 261.62 0)
       (effects (font (size 1.27 1.27)) hide)
     )
@@
   (symbol (lib_id "power:GND") (at 260.35 36.83 0) (unit 1)
     (in_bom yes) (on_board yes) (fields_autoplaced)
-    (property "Reference" "#PWR087" (id 0) (at 260.35 43.18 0)
+    (property "Reference" "#PWR089" (id 0) (at 260.35 43.18 0)
       (effects (font (size 1.27 1.27)) hide)
     )
@@
   (symbol (lib_id "power:GND") (at 289.56 49.53 0) (unit 1)
     (in_bom yes) (on_board yes) (fields_autoplaced)
-    (property "Reference" "#PWR090" (id 0) (at 289.56 55.88 0)
+    (property "Reference" "#PWR092" (id 0) (at 289.56 55.88 0)
       (effects (font (size 1.27 1.27)) hide)
     )
@@
   (symbol (lib_id "power:GND") (at 43.18 270.51 0) (unit 1)
     (in_bom yes) (on_board yes) (fields_autoplaced)
-    (property "Reference" "#PWR082" (id 0) (at 43.18 276.86 0)
+    (property "Reference" "#PWR083" (id 0) (at 43.18 276.86 0)
       (effects (font (size 1.27 1.27)) hide)
     )
@@
   (symbol (lib_id "power:GND") (at 306.07 41.91 0) (unit 1)
     (in_bom yes) (on_board yes) (fields_autoplaced)
-    (property "Reference" "#PWR091" (id 0) (at 306.07 48.26 0)
+    (property "Reference" "#PWR093" (id 0) (at 306.07 48.26 0)
       (effects (font (size 1.27 1.27)) hide)
     )
@@
   (symbol (lib_id "Regulator_Linear:AMS1117-3.3") (at 43.18 257.81 0) (unit 1)
     (in_bom yes) (on_board yes) (fields_autoplaced)
-    (property "Reference" "U19" (id 0) (at 43.18 250.19 0))
+    (property "Reference" "U18" (id 0) (at 43.18 250.19 0))
     (property "Value" "AMS1117-3.3" (id 1) (at 43.18 252.73 0))
     (property "Footprint" "Package_TO_SOT_SMD:SOT-223-3_TabPin2" (id 2) (at 43.18 252.73 0)
@@
   (symbol (lib_id "Connector_Generic:Conn_02x21_Odd_Even") (at 184.15 63.5 0) (unit 1)
     (in_bom yes) (on_board yes) (fields_autoplaced)
-    (property "Reference" "J9" (id 0) (at 185.42 31.75 0))
+    (property "Reference" "J8" (id 0) (at 185.42 31.75 0))
     (property "Value" "Conn_02x21_Odd_Even" (id 1) (at 185.42 34.29 0))
     (property "Footprint" "Connector_PinHeader_2.54mm:PinHeader_2x21_P2.54mm_Vertical" (id 2) (at 184.15 63.5 0)
@@
   (symbol (lib_id "Device:R") (at 240.03 144.78 0) (unit 1)
     (in_bom yes) (on_board yes) (fields_autoplaced)
-    (property "Reference" "R40" (id 0) (at 242.57 143.5099 0)
+    (property "Reference" "R48" (id 0) (at 242.57 143.5099 0)
       (effects (font (size 1.27 1.27)) (justify left))
     )
@@
   (symbol (lib_id "Device:R") (at 240.03 134.62 0) (unit 1)
     (in_bom yes) (on_board yes) (fields_autoplaced)
-    (property "Reference" "R37" (id 0) (at 242.57 133.3499 0)
+    (property "Reference" "R47" (id 0) (at 242.57 133.3499 0)
       (effects (font (size 1.27 1.27)) (justify left))
     )
@@
   (symbol (lib_id "power:GND") (at 337.82 43.18 0) (unit 1)
     (in_bom yes) (on_board yes) (fields_autoplaced)
-    (property "Reference" "#PWR093" (id 0) (at 337.82 49.53 0)
-      (effects (font (size 1.27 1.27)) hide)
-    )
+    (property "Reference" "#PWR095" (id 0) (at 337.82 49.53 0)
+      (effects (font (size 1.27 1.27)) hide)
+    )
